File: Hardware/motor_control_hat/00/motor_control_hat/motor_control_hat.kicad_sch (KiCad schematic)
At the start: 29 parts, among them P1 TB_1x2_5.08mm_RA, P10 X9254WR-04-N0SN, P11 X9254WR-04-N0SN, P12 X9254WR-04-N0SN, P13 X9254WR-04-N0SN, P5 X9254WR-04-N0SN, P6 X9254WR-04-N0SN, P7 X9254WR-04-N0SN, P8 X9254WR-04-N0SN, P9 X9254WR-04-N0SN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

Commit message: Connectors changed. New power distribution board
Parts:
- removed P10, P11, P12, P13, P5, P6, P7, P8, P9: X9254WR-04-N0SN, CustomConnectors:X9254WR-04-N0SN, symbol CustomConnectors:X9254WR-04-N0SN
- added J10, J11, J3, J4, J5, J6, J7, J8, J9: S4B-XH-A(LF)(SN), Connector_JST:JST_XH_S4B-XH-A_1x04_P2.50mm_Horizontal, symbol Connector_Generic:Conn_01x04
- TP1, U1: JLCPCB BOM (none) -> 0; LCSC (none) -> -
- TP2: renamed from TP4; JLCPCB BOM (none) -> 0; LCSC (none) -> -
- TP3: renamed from TP17; JLCPCB BOM (none) -> 0; LCSC (none) -> -
- renumbered P1 to J1
Connections:
- net +5V: now also J10.1 (Pin_1), J11.1 (Pin_1), J3.1 (Pin_1), J4.1 (Pin_1), J5.1 (Pin_1), J6.1 (Pin_1), J7.1 (Pin_1), J8.1 (Pin_1), J9.1 (Pin_1)
- net ENC1_PHA: now also J6.2 (Pin_2)
- net ENC1_PHB: now also J6.3 (Pin_3)
- net ENC2_PHA: now also J7.2 (Pin_2)
- net ENC2_PHB: now also J7.3 (Pin_3)
- net ENC3_PHA: now also J8.2 (Pin_2)
- net ENC3_PHB: now also J8.3 (Pin_3)
- net GND: now also J10.4 (Pin_4), J11.4 (Pin_4), J3.2 (Pin_2), J4.2 (Pin_2), J5.4 (Pin_4), J6.4 (Pin_4), J7.4 (Pin_4), J8.4 (Pin_4), J9.4 (Pin_4)
- net OC_IN_1: now also J3.3 (Pin_3)
- net OC_IN_2: now also J4.3 (Pin_3)
- net PWM_CH_1: now also J9.3 (Pin_3)
- net PWM_CH_2: now also J10.3 (Pin_3)
- net PWM_CH_3: now also J11.3 (Pin_3)
- net PWM_DIR_1: now also J9.2 (Pin_2)
- net PWM_DIR_2: now also J10.2 (Pin_2)
- net PWM_DIR_3: now also J11.2 (Pin_2)
- net USART3_RX: now also J5.2 (Pin_2)
- net USART3_TX: now also J5.3 (Pin_3)
Other:
- company: (none) -> Roobolabo
- title: (none) -> motro_control_hat
