Commit message: feat: imu sensor added
imu model & plugin (gazebo & rviz)

File: nomad200-ros2/src/model/urdf/nomad200/macros.xacro (robot description, xacro)
@@ -2,23 +2,24 @@
 <robot xmlns:xacro="http://www.ros.org/wiki/xacro">
     <xacro:macro name="link_wheel" params="name">
-        <link name="${name}">
-            <inertial>
-              <mass value="0.2"/>
-              <origin rpy="0 1.5707 1.5707" xyz="0 0 0"/>
-              <inertia ixx="0.000526666666667" ixy="0" ixz="0" iyy="0.000526666666667" iyz="0" izz="0.001"/>
-            </inertial>
-            <collision name="link_right_wheel_collision">
-              <origin rpy="0 1.5707 1.5707" xyz="0 0 0"/>
-              <geometry>
-                <cylinder length="0.04" radius="0.1"/>
-              </geometry>
-            </collision>
-            <visual name="${name}_visual">
-              <origin rpy="0 1.5707 1.5707" xyz="0 0 0"/>
-              <geometry>
-                <cylinder length="0.04" radius="0.1"/>
-              </geometry>
-            </visual>
-        </link>
+      <link name="${name}">
+          <inertial>
+            <mass value="0.2"/>
+            <origin rpy="0 1.5707 1.5707" xyz="0 0 0"/>
+            <inertia ixx="0.000526666666667" ixy="0" ixz="0" iyy="0.000526666666667" iyz="0" izz="0.001"/>
+           </inertial>
+           <collision name="${name}_collision">
+             <origin rpy="0 1.5707 1.5707" xyz="0 0 0"/>
+             <geometry>
+               <cylinder length="0.04" radius="0.1"/>
+             </geometry>
+           </collision>
+           <visual name="${name}_visual">
+             <origin rpy="0 1.5707 1.5707" xyz="0 0 0"/>
+             <geometry>
+               <cylinder length="0.04" radius="0.1"/>
+             </geometry>
+             <material name="Nomad/Blue"/>
+           </visual>
+      </link>
     </xacro:macro>
     <xacro:macro name="joint_wheel" params="name child origin_xyz">
@@ -32,3 +33,33 @@
       </joint>
     </xacro:macro>
+    <xacro:macro name="link_imu" params="name">
+      <link name="${name}">
+        <inertial>
+          <mass value="0.001" />
+          <origin xyz="0 0 0" rpy="0 0 0" />
+          <inertia ixx="0.00000015" ixy="0" ixz="0" iyy="0.00000015" iyz="0" izz="0.00000015" />
+        </inertial>
+        <collision  name="${name}_collision">
+          <origin xyz="0 0 0" rpy="0 0 0" />
+          <geometry>
+            <box size="0.02 0.02 0.02" />
+          </geometry>
+        </collision>
+        <visual  name="${name}_visual">
+          <origin xyz="0 0 0" rpy="0 0 0" />
+          <geometry>
+            <box size="0.02 0.02 0.02" />
+          </geometry>
+          <material name="Nomad/Green"/>
+        </visual>
+      </link>
+    </xacro:macro>
+    <xacro:macro name="joint_imu" params="name child origin_xyz rpy">
+      <joint name="${name}" type="fixed">
+        <origin xyz="${origin_xyz}" rpy="${rpy}" />
+        <child link="${child}" />
+        <parent link="link_chassis" />
+        <axis xyz="0 0 1" />
+      </joint>
+    </xacro:macro>
 </robot>

File: nomad200-ros2/src/model/urdf/nomad200/materials.xacro (robot description, xacro)
@@ -1,26 +1,26 @@
 <?xml version="1.0" ?>
 <robot>
-  <material name="black">
+  <material name="Nomad/Black">
     <color rgba="0.0 0.0 0.0 1.0"/>
   </material>
-  <material name="blue">
-    <color rgba="0.203125 0.23828125 0.28515625 1.0"/>
+  <material name="Nomad/Blue">
+    <color rgba="0.0 0.0 0.9 1.0"/>
   </material>
-  <material name="green">
+  <material name="Nomad/Green">
     <color rgba="0.0 0.8 0.0 1.0"/>
   </material>
-  <material name="grey">
+  <material name="Nomad/Grey">
     <color rgba="0.2 0.2 0.2 1.0"/>
   </material>
-  <material name="orange">
+  <material name="Nomad/Orange">
     <color rgba="1.0 0.423529411765 0.0392156862745 1.0"/>
   </material>
-  <material name="brown">
+  <material name="Nomad/Brown">
     <color rgba="0.870588235294 0.811764705882 0.764705882353 1.0"/>
   </material>
-  <material name="red">
-    <color rgba="0.80078125 0.12890625 0.1328125 1.0"/>
+  <material name="Nomad/Red">
+    <color rgba="0.9 0.0 0.0 1.0"/>
   </material>
-  <material name="white">
+  <material name="Nomad/White">
     <color rgba="1.0 1.0 1.0 1.0"/>
   </material>

File: nomad200-ros2/src/model/urdf/nomad200/robot.urdf.xacro (robot description, xacro)
@@ -25,5 +25,5 @@
         <cylinder radius="0.25" length="0.05"/>
       </geometry>
-      <material name="blue"/>
+      <material name="Nomad/Grey"/>
     </visual>
     <!-- caster front -->
@@ -49,4 +49,5 @@
         <sphere radius="0.05"/>
       </geometry>
+      <material name="Nomad/Black"/>
     </visual>
   </link>
@@ -57,3 +58,6 @@
   <xacro:link_wheel name="link_left_wheel" />
   <xacro:joint_wheel name="joint_left_wheel" child="link_left_wheel" origin_xyz="-0.05 -0.15 0" />
+  <!-- imu -->
+  <xacro:link_imu name="link_sensor_imu" />
+  <xacro:joint_imu name="joint_sensor_imu" child="link_sensor_imu" origin_xyz="-0.1 0 0.05" rpy="0 0 0" />
 </robot>
