Commit message: Synchro-drive controller created

File: Software/nomad_ros2/nomad_robot/description/gazebo_control.xacro (robot description, xacro)
@@ -14,8 +14,20 @@
       <state_interface name="position" />
     </joint>
+    <joint name="left_steering_joint">
+      <command_interface name="position" />
+    </joint>
+    <joint name="left_wheel_joint">
+      <command_interface name="velocity" />
+    </joint>
+    <joint name="right_wheel_joint">
+      <command_interface name="velocity" />
+    </joint>
+    <joint name="right_steering_joint">
+      <command_interface name="position" />
+    </joint>
   </ros2_control>
   <gazebo>
     <plugin filename="libgazebo_ros2_control.so" name="gazebo_ros2_control">
-      <parameters>$(find gazebo_ros2_control_demos)/config/tricycle_drive_controller.yaml</parameters>
+      <parameters>/mnt/c/Workspace/repositories/NomadRehab/Software/nomad_ros2/nomad_robot/config/nomad_drive_controller.yaml</parameters>
     </plugin>
   </gazebo>

File: Software/nomad_ros2/nomad_robot/description/robot_wheels.xacro (robot description, xacro)
@@ -9,6 +9,6 @@
   <xacro:property name="wheel_thickness" value="0.08"/>
   <xacro:property name="wheel_mass" value="0.05"/>
-  <xacro:property name="base_mass" value="0.05"/>
-  <xacro:property name="base_thickness" value="0.1"/>
+  <xacro:property name="base_mass" value="1"/>
+  <xacro:property name="base_thickness" value="0.5"/>
   <xacro:include filename="inertial_macros.xacro"/>
   <link name="base_link" />

Commit message: Hardware interface working!

File: Software/nomad_ros2/nomad_robot/description/gazebo_control.xacro (robot description, xacro)
@@ -12,17 +12,16 @@
       <command_interface name="velocity" />
       <state_interface name="velocity" />
+    </joint>
+    <joint name="left_steering_joint">
       <state_interface name="position" />
     </joint>
-    <joint name="left_steering_joint">
-      <command_interface name="position" />
-    </joint>
     <joint name="left_wheel_joint">
-      <command_interface name="velocity" />
+      <state_interface name="velocity" />
     </joint>
     <joint name="right_wheel_joint">
-      <command_interface name="velocity" />
+      <state_interface name="velocity" />
     </joint>
     <joint name="right_steering_joint">
-      <command_interface name="position" />
+      <state_interface name="position" />
     </joint>
   </ros2_control>

File: Software/nomad_ros2/nomad_robot/description/robot.urdf.xacro (robot description, xacro)
@@ -3,4 +3,4 @@
     <xacro:include filename="materials.xacro"/>
     <xacro:include filename="robot_wheels.xacro"/>
-    <xacro:include filename="gazebo_control.xacro"/>
+    <xacro:include filename="robot_control.xacro"/>
 </robot>

File: Software/nomad_ros2/nomad_robot/description/robot_wheels.xacro (robot description, xacro)
@@ -40,4 +40,32 @@
     <child link="chassis" />
   </joint>
+  <!-- rotatory base  -->
+  <link name="rotatory_base">
+    <collision>
+      <origin xyz="0 0 0" rpy="0 0 0" />
+      <geometry>
+        <cylinder length="${base_thickness}" radius="${base_radius}" />
+      </geometry>
+    </collision>
+    <visual>
+      <origin xyz="0 0 0" rpy="0 0 0" />
+      <geometry>
+        <cylinder length="${base_thickness}" radius="${base_radius}" />
+      </geometry>
+      <material name="Orange" />
+    </visual>
+    <xacro:inertial_cylinder mass="${base_mass}" length="${base_thickness}" radius="${base_radius}">
+      <origin xyz="0 0 0" rpy="0 0 0"/>
+    </xacro:inertial_cylinder>
+  </link>
+  <gazebo reference="rotatory_base">
+    <material>Gazebo/Orange</material>
+  </gazebo>
+  <joint name="rotatory_base_joint" type="continuous">
+    <origin xyz="0 0 ${wheel_radius*2}" rpy="0 0 0" />
+    <parent link="chassis" />
+    <child link="rotatory_base" />
+    <axis xyz="0 0 1"/>
+  </joint>
   <!-- left Steering Link -->
   <link name="left_steering_link">

Commit message: Transform issue solved!

File: Software/nomad_ros2/nomad_robot/description/gazebo_control.xacro (robot description, xacro)
@@ -5,28 +5,38 @@
       <plugin>gazebo_ros2_control/GazeboSystem</plugin>
     </hardware>
-    <joint name="steering_joint">
-      <command_interface name="position" />
-      <state_interface name="position" />
-    </joint>
-    <joint name="traction_joint">
-      <command_interface name="velocity" />
-      <state_interface name="velocity" />
+    <!-- Base joint -->
+    <joint name="left_wheel_joint">
+      <state_interface name="velocity"/>
+      <state_interface name="position"/>
     </joint>
     <joint name="left_steering_joint">
-      <state_interface name="position" />
-    </joint>
-    <joint name="left_wheel_joint">
-      <state_interface name="velocity" />
+      <state_interface name="position"/>
     </joint>
     <joint name="right_wheel_joint">
-      <state_interface name="velocity" />
+      <state_interface name="velocity"/>
+      <state_interface name="position"/>
     </joint>
     <joint name="right_steering_joint">
-      <state_interface name="position" />
+      <state_interface name="position"/>
+    </joint>
+    <!-- Base joint -->
+    <joint name="traction_joint">
+      <command_interface name="velocity"/>
+      <state_interface name="velocity"/>
+      <state_interface name="position"/>
+    </joint>
+    <joint name="rotatory_base_joint">
+      <command_interface name="position"/>
+      <state_interface name="position"/>
+    </joint>
+    <!-- Steering joint -->
+    <joint name="steering_joint">
+      <command_interface name="position"/>
+      <state_interface name="position"/>
     </joint>
   </ros2_control>
   <gazebo>
     <plugin filename="libgazebo_ros2_control.so" name="gazebo_ros2_control">
-      <parameters>/mnt/c/Workspace/repositories/NomadRehab/Software/nomad_ros2/nomad_robot/config/nomad_drive_controller.yaml</parameters>
+      <parameters>$(find nomad_robot)/config/nomad_drive_controller.yaml</parameters>
     </plugin>
   </gazebo>

File: Software/nomad_ros2/nomad_robot/description/robot.urdf.xacro (robot description, xacro)
@@ -3,4 +3,9 @@
     <xacro:include filename="materials.xacro"/>
     <xacro:include filename="robot_wheels.xacro"/>
-    <xacro:include filename="robot_control.xacro"/>
+    <xacro:if value="$(arg use_ros2_control)">
+      <xacro:include filename="robot_control.xacro" />
+    </xacro:if>
+    <xacro:unless value="$(arg use_ros2_control)">
+        <xacro:include filename="gazebo_control.xacro" />
+    </xacro:unless>
 </robot>

File: Software/nomad_ros2/nomad_robot/description/robot_control.xacro (robot description, xacro)
@@ -4,5 +4,5 @@
     <hardware>
       <plugin>nomad_hardware_interface/NomadHardware</plugin>
-      <param name="emulate">0</param>
+      <param name="emulate">1</param>
       <!-- communication parameters -->
       <param name="serial_port">/dev/ttyUSB0</param>
@@ -39,36 +39,33 @@
     </hardware>
     <!-- Base joint -->
+    <joint name="left_wheel_joint">
+      <state_interface name="velocity"/>
+      <state_interface name="position"/>
+    </joint>
+    <joint name="left_steering_joint">
+      <state_interface name="position"/>
+    </joint>
+    <joint name="right_wheel_joint">
+      <state_interface name="velocity"/>
+      <state_interface name="position"/>
+    </joint>
+    <joint name="right_steering_joint">
+      <state_interface name="position"/>
+    </joint>
     <!-- Base joint -->
     <joint name="traction_joint">
-      <command_interface name="velocity" />
-      <state_interface name="velocity" />
+      <command_interface name="velocity"/>
+      <state_interface name="velocity"/>
+      <state_interface name="position"/>
     </joint>
     <joint name="rotatory_base_joint">
-      <command_interface name="position" />
-      <state_interface name="position" />
+      <command_interface name="position"/>
+      <state_interface name="position"/>
     </joint>
     <!-- Steering joint -->
     <joint name="steering_joint">
-      <command_interface name="position" />
-      <state_interface name="position" />
-    </joint>
-    <!-- Back wheels joints -->
-    <joint name="left_steering_joint">
-      <state_interface name="position" />
-    </joint>
-    <joint name="left_wheel_joint">
-      <state_interface name="velocity" />
-    </joint>
-    <joint name="right_wheel_joint">
-      <state_interface name="velocity" />
-    </joint>
-    <joint name="right_steering_joint">
-      <state_interface name="position" />
+      <command_interface name="position"/>
+      <state_interface name="position"/>
     </joint>
   </ros2_control>
-  <gazebo>
-    <plugin filename="libgazebo_ros2_control.so" name="gazebo_ros2_control">
-      <parameters>/mnt/c/Workspace/repositories/NomadRehab/Software/nomad_ros2/nomad_robot/config/nomad_drive_controller.yaml</parameters>
-    </plugin>
-  </gazebo>
 </robot>

File: Software/nomad_ros2/nomad_robot/description/robot_wheels.xacro (robot description, xacro)
@@ -35,4 +35,129 @@
     <material>Gazebo/Orange</material>
   </gazebo>
+  <!-- rotatory base  -->
+  <link name="rotatory_base">
+    <collision>
+      <origin xyz="0 0 0" rpy="0 0 0" />
+      <geometry>
+        <cylinder length="${base_thickness}" radius="${base_radius}" />
+      </geometry>
+    </collision>
+    <visual>
+      <origin xyz="0 0 0" rpy="0 0 0" />
+      <geometry>
+        <cylinder length="${base_thickness}" radius="${base_radius}" />
+      </geometry>
+      <material name="Orange" />
+    </visual>
+    <xacro:inertial_cylinder mass="${base_mass}" length="${base_thickness}" radius="${base_radius}">
+      <origin xyz="0 0 0" rpy="0 0 0"/>
+    </xacro:inertial_cylinder>
+  </link>
+  <gazebo reference="rotatory_base">
+    <material>Gazebo/Orange</material>
+  </gazebo>
+  <!-- left Steering Link -->
+  <link name="left_steering_link">
+    <visual>
+      <geometry>
+        <box size="0.01 0.01 0.01" />
+      </geometry>
+      <material name="Black" />
+    </visual>
+    <inertial>
+      <origin xyz="0 0 0" rpy="0 0 0" />
+      <mass value="0.005" />
+      <inertia ixx="0.1" ixy="0.0" ixz="0.0" iyy="0.1" iyz="0.0" izz="0.1" />
+    </inertial>
+  </link>
+  <!-- left wheel Link -->
+  <link name="left_wheel_link">
+    <collision>
+      <geometry>
+        <cylinder length="${wheel_thickness}" radius="${wheel_radius}" />
+      </geometry>
+    </collision>
+    <visual>
+      <geometry>
+        <cylinder length="${wheel_thickness}" radius="${wheel_radius}"/>
+      </geometry>
+      <material name="Black" />
+    </visual>
+    <xacro:inertial_cylinder mass="${wheel_mass}" length="${wheel_thickness}" radius="${wheel_radius}">
+      <origin xyz="0 0 0" rpy="0 0 0"/>
+    </xacro:inertial_cylinder>
+  </link>
+  <gazebo reference="left_wheel_link">
+    <material>Gazebo/Black</material>
+  </gazebo>
+  <!-- right Steering Link -->
+    <link name="right_steering_link">
+    <visual>
+      <geometry>
+        <box size="0.01 0.01 0.01" />
+      </geometry>
+      <material name="Black" />
+    </visual>
+    <inertial>
+      <origin xyz="0 0 0" rpy="0 0 0" />
+      <mass value="0.005" />
+      <inertia ixx="0.1" ixy="0.0" ixz="0.0" iyy="0.1" iyz="0.0" izz="0.1" />
+    </inertial>
+  </link>
+  <!-- right wheel Link -->
+  <link name="right_wheel_link">
+    <collision>
+      <geometry>
+        <cylinder length="${wheel_thickness}" radius="${wheel_radius}"/>
+      </geometry>
+    </collision>
+    <visual>
+      <geometry>
+        <cylinder length="${wheel_thickness}" radius="${wheel_radius}"/>
+      </geometry>
+      <material name="Black" />
+    </visual>
+    <xacro:inertial_cylinder mass="${wheel_mass}" length="${wheel_thickness}" radius="${wheel_radius}">
+      <origin xyz="0 0 0" rpy="0 0 0"/>
+    </xacro:inertial_cylinder>
+  </link>
+  <gazebo reference="right_wheel_link">
+    <material>Gazebo/Black</material>
+  </gazebo>
+  <!-- Steering Link -->
+  <link name="steering_link">
+    <visual>
+      <geometry>
+        <box size="0.01 0.01 0.01" />
+      </geometry>
+      <material name="Black" />
+    </visual>
+    <inertial>
+      <origin xyz="0 0 0" rpy="0 0 0" />
+      <mass value="0.005" />
+      <inertia ixx="0.1" ixy="0.0" ixz="0.0" iyy="0.1" iyz="0.0" izz="0.1" />
+    </inertial>
+  </link>
+  <!-- traction wheel link -->
+  <link name="wheel_front_link">
+    <collision>
+      <geometry>
+        <cylinder length="${wheel_thickness}" radius="${wheel_radius}"/>
+      </geometry>
+    </collision>
+    <visual>
+      <geometry>
+        <cylinder length="${wheel_thickness}" radius="${wheel_radius}"/>
+      </geometry>
+      <material name="Black" />
+    </visual>
+    <xacro:inertial_cylinder mass="${wheel_mass}" length="${wheel_thickness}" radius="${wheel_radius}">
+      <origin xyz="0 0 0" rpy="0 0 0"/>
+    </xacro:inertial_cylinder>
+  </link>
+  <gazebo reference="wheel_front_link">
+    <material>Gazebo/Black</material>
+  </gazebo>
+  <!-- Joints -->
   <joint name="chassis_joint" type="fixed">
     <origin xyz="0 0 ${wheel_radius*2}" rpy="0 0 0" />
@@ -40,26 +165,4 @@
     <child link="chassis" />
   </joint>
-  <!-- rotatory base  -->
-  <link name="rotatory_base">
-    <collision>
-      <origin xyz="0 0 0" rpy="0 0 0" />
-      <geometry>
-        <cylinder length="${base_thickness}" radius="${base_radius}" />
-      </geometry>
-    </collision>
-    <visual>
-      <origin xyz="0 0 0" rpy="0 0 0" />
-      <geometry>
-        <cylinder length="${base_thickness}" radius="${base_radius}" />
-      </geometry>
-      <material name="Orange" />
-    </visual>
-    <xacro:inertial_cylinder mass="${base_mass}" length="${base_thickness}" radius="${base_radius}">
-      <origin xyz="0 0 0" rpy="0 0 0"/>
-    </xacro:inertial_cylinder>
-  </link>
-  <gazebo reference="rotatory_base">
-    <material>Gazebo/Orange</material>
-  </gazebo>
   <joint name="rotatory_base_joint" type="continuous">
     <origin xyz="0 0 ${wheel_radius*2}" rpy="0 0 0" />
@@ -68,112 +171,4 @@
     <axis xyz="0 0 1"/>
   </joint>
-  <!-- left Steering Link -->
-  <link name="left_steering_link">
-    <visual>
-      <geometry>
-        <box size="0.01 0.01 0.01" />
-      </geometry>
-      <material name="Black" />
-    </visual>
-    <inertial>
-      <origin xyz="0 0 0" rpy="0 0 0" />
-      <mass value="0.005" />
-      <inertia ixx="0.1" ixy="0.0" ixz="0.0" iyy="0.1" iyz="0.0" izz="0.1" />
-    </inertial>
-  </link>
-  <joint name="left_steering_joint" type="continuous">
-    <origin xyz="${-wheel_wheelbase/2} ${wheel_track/2} ${-wheel_radius}" rpy="0 0 0" />
-    <parent link="chassis" />
-    <child link="left_steering_link" />
-    <axis xyz="0 0 1" />
-  </joint>
-  <!-- left wheel Link -->
-  <link name="left_wheel">
-    <collision>
-      <geometry>
-        <cylinder length="${wheel_thickness}" radius="${wheel_radius}" />
-      </geometry>
-    </collision>
-    <visual>
-      <geometry>
-        <cylinder length="${wheel_thickness}" radius="${wheel_radius}"/>
-      </geometry>
-      <material name="Black" />
-    </visual>
-    <xacro:inertial_cylinder mass="${wheel_mass}" length="${wheel_thickness}" radius="${wheel_radius}">
-      <origin xyz="0 0 0" rpy="0 0 0"/>
-    </xacro:inertial_cylinder>
-  </link>
-  <gazebo reference="left_wheel">
-    <material>Gazebo/Black</material>
-  </gazebo>
-  <joint name="left_wheel_joint" type="continuous">
-    <origin xyz="0 0 0" rpy="-1.57 0 0" />
-    <parent link="left_steering_link" />
-    <child link="left_wheel" />
-    <axis xyz="0 0 1" />
-    <dynamics damping="0.2" />
-  </joint>
-  <!-- right Steering Link -->
-    <link name="right_steering_link">
-    <visual>
-      <geometry>
-        <box size="0.01 0.01 0.01" />
-      </geometry>
-      <material name="Black" />
-    </visual>
-    <inertial>
-      <origin xyz="0 0 0" rpy="0 0 0" />
-      <mass value="0.005" />
-      <inertia ixx="0.1" ixy="0.0" ixz="0.0" iyy="0.1" iyz="0.0" izz="0.1" />
-    </inertial>
-  </link>
-  <joint name="right_steering_joint" type="continuous">
-    <origin xyz="${-wheel_wheelbase/2} ${-wheel_track/2} ${-wheel_radius}" rpy="0 0 0" />
-    <parent link="chassis" />
-    <child link="right_steering_link" />
-    <axis xyz="0 0 1" />
-  </joint>
-  <!-- right wheel Link -->
-  <link name="right_wheel">
-    <collision>
-      <geometry>
-        <cylinder length="${wheel_thickness}" radius="${wheel_radius}"/>
-      </geometry>
-    </collision>
-    <visual>
-      <geometry>
-        <cylinder length="${wheel_thickness}" radius="${wheel_radius}"/>
-      </geometry>
-      <material name="Black" />
-    </visual>
-    <xacro:inertial_cylinder mass="${wheel_mass}" length="${wheel_thickness}" radius="${wheel_radius}">
-      <origin xyz="0 0 0" rpy="0 0 0"/>
-    </xacro:inertial_cylinder>
-  </link>
-  <gazebo reference="right_wheel">
-    <material>Gazebo/Black</material>
-  </gazebo>
-  <joint name="right_wheel_joint" type="continuous">
-    <origin xyz="0 0 0" rpy="-1.57 0 0" />
-    <parent link="right_steering_link" />
-    <child link="right_wheel" />
-    <axis xyz="0 0 1" />
-    <dynamics damping="0.2" />
-  </joint>
-  <!-- Steering Link -->
-  <link name="steering_link">
-    <visual>
-      <geometry>
-        <box size="0.01 0.01 0.01" />
-      </geometry>
-      <material name="Black" />
-    </visual>
-    <inertial>
-      <origin xyz="0 0 0" rpy="0 0 0" />
-      <mass value="0.005" />
-      <inertia ixx="0.1" ixy="0.0" ixz="0.0" iyy="0.1" iyz="0.0" izz="0.1" />
-    </inertial>
-  </link>
   <joint name="steering_joint" type="continuous">
     <origin xyz="${wheel_wheelbase/2} 0 ${-wheel_radius}" rpy="0 0 0" />
@@ -182,24 +177,4 @@
     <axis xyz="0 0 1" />
   </joint>
-  <!-- traction wheel link -->
-  <link name="wheel_front_link">
-    <collision>
-      <geometry>
-        <cylinder length="${wheel_thickness}" radius="${wheel_radius}"/>
-      </geometry>
-    </collision>
-    <visual>
-      <geometry>
-        <cylinder length="${wheel_thickness}" radius="${wheel_radius}"/>
-      </geometry>
-      <material name="Black" />
-    </visual>
-    <xacro:inertial_cylinder mass="${wheel_mass}" length="${wheel_thickness}" radius="${wheel_radius}">
-      <origin xyz="0 0 0" rpy="0 0 0"/>
-    </xacro:inertial_cylinder>
-  </link>
-  <gazebo reference="wheel_front_link">
-    <material>Gazebo/Black</material>
-  </gazebo>
   <joint name="traction_joint" type="continuous">
     <parent link="steering_link" />
@@ -208,3 +183,27 @@
     <axis xyz="0 0 1" />
   </joint>
+  <joint name="left_steering_joint" type="continuous">
+    <origin xyz="${-wheel_wheelbase/2} ${wheel_track/2} ${-wheel_radius}" rpy="0 0 0" />
+    <parent link="chassis" />
+    <child link="left_steering_link" />
+    <axis xyz="0 0 1" />
+  </joint>
+  <joint name="right_steering_joint" type="continuous">
+    <origin xyz="${-wheel_wheelbase/2} ${-wheel_track/2} ${-wheel_radius}" rpy="0 0 0" />
+    <parent link="chassis" />
+    <child link="right_steering_link" />
+    <axis xyz="0 0 1" />
+  </joint>
+  <joint name="left_wheel_joint" type="continuous">
+    <origin xyz="0 0 0" rpy="-1.57 0 0" />
+    <parent link="left_steering_link" />
+    <child link="left_wheel_link" />
+    <axis xyz="0 0 1" />
+  </joint>
+  <joint name="right_wheel_joint" type="continuous">
+    <origin xyz="0 0 0" rpy="-1.57 0 0" />
+    <parent link="right_steering_link" />
+    <child link="right_wheel_link" />
+    <axis xyz="0 0 1" />
+  </joint>
 </robot>
