Commit message: Added  sonar and IR description

File: Software/nomad_ros2/nomad_robot/description/materials.xacro (robot description, xacro)
@@ -2,4 +2,7 @@
   <material name="Black">
     <color rgba="0 0 0 1" />
+  </material>
+  <material name="red">
+    <color rgba="1 0 0 1" />
   </material>
   <material name="Grey">

File: Software/nomad_ros2/nomad_robot/description/robot.urdf.xacro (robot description, xacro)
@@ -3,4 +3,6 @@
     <xacro:include filename="materials.xacro"/>
     <xacro:include filename="robot_wheels.xacro"/>
+    <xacro:include filename="sonar.xacro"/>
+    <xacro:include filename="infrarated.xacro"/>
     <xacro:if value="$(arg use_ros2_control)">
       <xacro:include filename="robot_control.xacro" />
